File: Digital_Outputs.kicad_sch (KiCad schematic)
At the start: 5 parts, among them K1 G2RL-1, K2 G2RL-1, U8 ULN2003A

Commit message: Трассировка питания и цифровых входов-выходов
Connections:
- net K1_A2: now also U8.15 (O2); no longer U8.16 (O1)
- net K2_A2: now also U8.16 (O1); no longer U8.15 (O2)
Changed lines of the file:
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@@
+	(wire
+		(pts
+			(xy 163.83 68.58) (xy 189.23 68.58)
+		)
+		(stroke
+			(width 0)
+			(type default)
+		)
+	)
 	(wire
 		(pts
@@
 	(wire
 		(pts
-			(xy 163.83 68.58) (xy 189.23 68.58)
+			(xy 129.54 77.47) (xy 134.62 77.47)
 		)
 		(stroke
@@
 		(pts
 			(xy 166.37 86.36) (xy 177.8 86.36)
-		)
-		(stroke
-			(width 0)
-			(type default)
-		)
-	)
-	(wire
-		(pts
-			(xy 129.54 77.47) (xy 134.62 77.47)
 		)
 		(stroke
@@
 	)
 	(label "K1_A2"
-		(at 134.62 74.93 0)
+		(at 134.62 77.47 0)
 		(effects
 			(font
@@
 	)
 	(label "K2_A2"
-		(at 134.62 77.47 0)
-		(effects
-			(font
+		(at 134.62 74.93 0)
+		(effects
+			(font
