File: Mini_Control_24v.kicad_sch (KiCad schematic)
At the start: 19 parts, among them J1 Screw_Terminal_01x02, J2 Screw_Terminal_01x04, J3 Screw_Terminal_01x04, J4 Screw_Terminal_01x03, J5 Screw_Terminal_01x03, J6 ВН-20, J8 Screw_Terminal_01x02, U1 STM32F051C8Tx

Commit message: Трассировка питания и цифровых входов-выходов
Parts:
- J4, J5: footprint TerminalBlock_Phoenix:TerminalBlock_Phoenix_PT-1,5-3-5.0-H_1x03_P5.00mm_Horizontal -> Connector_Phoenix_MSTB:PhoenixContact_MSTBA_2,5_3-G-5,08_1x03_P5.08mm_Horizontal
Changed lines of the file:
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@@
 	(wire
 		(pts
-			(xy 194.31 63.5) (xy 186.69 63.5)
+			(xy 194.31 67.31) (xy 186.69 67.31)
 		)
 		(stroke
@@
 	(wire
 		(pts
-			(xy 194.31 67.31) (xy 194.31 63.5)
-		)
-		(stroke
-			(width 0)
-			(type default)
-		)
-	)
-	(wire
-		(pts
 			(xy 213.36 121.92) (xy 229.87 121.92)
 		)
@@
 	)
 	(label "+24V"
-		(at 186.69 63.5 0)
+		(at 186.69 67.31 0)
 		(effects
 			(font
@@
 			)
 		)
-		(property "Footprint" "TerminalBlock_Phoenix:TerminalBlock_Phoenix_PT-1,5-3-5.0-H_1x03_P5.00mm_Horizontal"
+		(property "Footprint" "Connector_Phoenix_MSTB:PhoenixContact_MSTBA_2,5_3-G-5,08_1x03_P5.08mm_Horizontal"
 			(at 233.68 52.07 0)
 			(hide yes)
@@
 			)
 		)
-		(property "Footprint" "TerminalBlock_Phoenix:TerminalBlock_Phoenix_PT-1,5-3-5.0-H_1x03_P5.00mm_Horizontal"
+		(property "Footprint" "Connector_Phoenix_MSTB:PhoenixContact_MSTBA_2,5_3-G-5,08_1x03_P5.08mm_Horizontal"
 			(at 233.68 62.23 0)
 			(hide yes)
